Commit message: fix: cut all 'eureka_simulation' mentions

File: description/sensors/all_sensors.urdf.xacro (robot description, xacro)
@@ -19,12 +19,12 @@
 <robot name="all_sensors" xmlns:xacro="http://www.ros.org/wiki/xacro">
   <!-- Imu -->
-  <xacro:include filename="$(find eureka_simulation)/description/sensors/imu.urdf.xacro" />
+  <xacro:include filename="$(find universal_simulation)/description/sensors/imu.urdf.xacro" />
   <!-- Hokuyo -->
-  <xacro:include filename="$(find eureka_simulation)/description/sensors/hokuyo.urdf.xacro" />
+  <xacro:include filename="$(find universal_simulation)/description/sensors/hokuyo.urdf.xacro" />
   <!-- Xtion -->
-  <xacro:include filename="$(find eureka_simulation)/description/sensors/asus_xtion.urdf.xacro" />
+  <xacro:include filename="$(find universal_simulation)/description/sensors/asus_xtion.urdf.xacro" />
   <!-- Realsense d415 -->
-  <xacro:include filename="$(find eureka_simulation)/description/sensors/realsense_d415.urdf.xacro" />
+  <xacro:include filename="$(find universal_simulation)/description/sensors/realsense_d415.urdf.xacro" />
   <!-- GPS -->
-  <xacro:include filename="$(find eureka_simulation)/description/sensors/gps.urdf.xacro" />
+  <xacro:include filename="$(find universal_simulation)/description/sensors/gps.urdf.xacro" />
 </robot>

File: description/sensors/asus_xtion.urdf.xacro (robot description, xacro)
@@ -30,5 +30,5 @@
         <origin rpy="${math_pi_over_2} 0 ${math_pi_over_2}" xyz="0 0 0"/>
         <geometry>
-          <mesh filename="file://$(find eureka_simulation)/meshes/sensors/asus_xtion/asus_xtion_pro_live.dae" scale="0.001 0.001 0.001"/>
+          <mesh filename="file://$(find universal_simulation)/meshes/sensors/asus_xtion/asus_xtion_pro_live.dae" scale="0.001 0.001 0.001"/>
         </geometry>
       </visual>
@@ -36,5 +36,5 @@
         <origin rpy="${math_pi_over_2} 0 ${math_pi_over_2}" xyz="0 0 0"/>
         <geometry>
-          <mesh filename="file://$(find eureka_simulation)/meshes/sensors/asus_xtion/asus_xtion_pro_live.dae" scale="0.001 0.001 0.001"/>
+          <mesh filename="file://$(find universal_simulation)/meshes/sensors/asus_xtion/asus_xtion_pro_live.dae" scale="0.001 0.001 0.001"/>
         </geometry>
       </collision>

File: description/sensors/hokuyo.urdf.xacro (robot description, xacro)
@@ -34,5 +34,5 @@
         <origin xyz="0 0 -0.05" rpy="0 0 0"/>
         <geometry>
-            <mesh filename="file://$(find eureka_simulation)/meshes/sensors/hokuyo/hokuyo_ust_20lx.dae"/>
+            <mesh filename="file://$(find universal_simulation)/meshes/sensors/hokuyo/hokuyo_ust_20lx.dae"/>
         </geometry>
       </visual>
